File: nixie_driver/nixie_driver.kicad_sch (KiCad schematic)
At the start: 0 parts

Commit message: redoing stuff
Parts:
- added 1 (x4): ~, Nixie_Tube_Socket_Eagle_Library:NIXIE_TUBE_SOCKET, symbol 2026-04-08_05-56-20:NIXIE_TUBE_SOCKET
- added C1, C2, C3, C4: 100nF, symbol Device:C_US
- added C5: 10uF, symbol Device:C_US
- added C6: 47uF, symbol Device:C_US
- added C7: 10uF/250V, symbol Device:C_US
- added J1: USB_B_Micro, symbol Connector:USB_B_Micro
- added J2: GPIO, symbol Connector:Conn_01x16_Pin
- added J3: HV_TEST, symbol Connector:Conn_01x02_Pin
- added J4: Screw_Terminal_01x02, symbol Connector:Screw_Terminal_01x02
- added R1, R2, R3, R4: 12k,1W, symbol Device:R
- added U1, U2, U3, U4: SN74141N, SN74141N:DIP762W46P254L2134H508Q16, symbol SN74141N:SN74141N

Commit message: imports
Parts:
- added J5, J6, J7, J8: Conn_01x08_Socket, symbol Connector:Conn_01x08_Socket
Other:
- note added: "170V"
- moved on the sheet: J1, J4, R1, R2, R3, R4

Commit message: fixed deisgn
Parts:
- removed 1 (x4): ~, Nixie_Tube_Socket_Eagle_Library:NIXIE_TUBE_SOCKET, symbol 2026-04-08_05-56-20:NIXIE_TUBE_SOCKET
- removed J5, J6, J7, J8: Conn_01x08_Socket, symbol Connector:Conn_01x08_Socket
- removed R1, R2, R3, R4: 12k,1W, symbol Device:R
- added J10, J11, J12, J9: Screw_Terminal_01x02, symbol Connector:Screw_Terminal_01x02
- added J5, J6, J7, J8: Conn_01x11_Pin, Connector_PinSocket_2.54mm:PinSocket_1x11_P2.54mm_Vertical, symbol Connector:Conn_01x11_Pin

Commit message: mostly done
Parts:
- removed C5: 10uF, symbol Device:C_US
- removed C6: 47uF, symbol Device:C_US
- added J13: USB_B_Micro, symbol Connector:USB_B_Micro
Connections:
- net GND: now reaches U1.12 (GND)
- net GND: now also J10.1 (Pin_1), J11.1 (Pin_1), J12.1 (Pin_1), J4.1 (Pin_1), J9.1 (Pin_1), U2.12 (GND), U3.12 (GND), U4.12 (GND)
- net U1_A: now reaches U1.3 (A)
- net U1_A: now also J2.1 (Pin_1)
- net U1_D: now reaches U1.4 (D)
- net U1_D: now also J2.4 (Pin_4)
- net at U1.5 (VCC): now also C1.2
- net U1_B: now reaches U1.6 (B)
- net U1_B: now also J2.2 (Pin_2)
- net U1_C: now reaches U1.7 (C)
- net U1_C: now also J2.3 (Pin_3)
- net 5V: now reaches C1.1
- net 5V: now also C2.1, C3.1, C4.1, J1.1 (VBUS), J13.1 (VBUS)
- net at J3.1 (Pin_1): now also C7.2, J10.2 (Pin_2), J11.2 (Pin_2), J12.2 (Pin_2), J9.2 (Pin_2)
- net at J1.2 (D-): now also J13.2 (D-)
- net at J1.3 (D+): now also J13.3 (D+)
- net at J1.4 (ID): now also J13.4 (ID)
- net at J1.5 (GND): now also J13.5 (GND)
- net at J1.6 (Shield): now also J13.6 (Shield)
- net 170V: now reaches C7.1
- net 170V: now also J4.2 (Pin_2)
- net U2_A: now reaches U2.3 (A)
- net U2_A: now also J2.5 (Pin_5)
- net U2_D: now reaches U2.4 (D)
- net U2_D: now also J2.8 (Pin_8)
- net at U2.5 (VCC): now also C2.2
- net U2_B: now reaches U2.6 (B)
- net U2_B: now also J2.6 (Pin_6)
- net U2_C: now reaches U2.7 (C)
- net U2_C: now also J2.7 (Pin_7)
- net at C3.2: now also U3.5 (VCC)
- net U3_B: now reaches J2.10 (Pin_10)
- net U3_B: now also U3.6 (B)
- net U3_C: now reaches J2.11 (Pin_11)
- net U3_C: now also U3.7 (C)
- net U3_D: now reaches J2.12 (Pin_12)
- net U3_D: now also U3.4 (D)
- net U4_A: now reaches J2.13 (Pin_13)
- net U4_A: now also U4.3 (A)
- net U4_B: now reaches J2.14 (Pin_14)
- net U4_B: now also U4.6 (B)
- net U4_C: now reaches J2.15 (Pin_15)
- net U4_C: now also U4.7 (C)
- net U4_D: now reaches J2.16 (Pin_16)
- net U4_D: now also U4.4 (D)
- net U3_A: now reaches J2.9 (Pin_9)
- net U3_A: now also U3.3 (A)
- net at U4.5 (VCC): now also C4.2
Other:
- note removed: "170V"
- moved on the sheet: C1, C2, C3, C4, C7, J10, J11, J12, J2, J3, J4, J5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

Commit message: more label
Connections:
- net GND: now also J1.5 (GND), J13.5 (GND), J5.11 (Pin_11), J6.11 (Pin_11), J7.11 (Pin_11), J8.11 (Pin_11)
- net U1_8: now reaches U1.1 (8)
- net U1_8: now also J5.9 (Pin_9)
- net U1_7: now reaches U1.10 (7)
- net U1_7: now also J5.8 (Pin_8)
- net U1_6: now reaches U1.11 (6)
- net U1_6: now also J5.7 (Pin_7)
- net U1_4: now reaches U1.13 (4)
- net U1_4: now also J5.5 (Pin_5)
- net U1_5: now reaches U1.14 (5)
- net U1_5: now also J5.6 (Pin_6)
- net U1_1: now reaches U1.15 (1)
- net U1_1: now also J5.2 (Pin_2)
- net U1_0: now reaches U1.16 (0)
- net U1_0: now also J5.1 (Pin_1)
- net U1_9: now reaches U1.2 (9)
- net U1_9: now also J5.10 (Pin_10)
- net U1_2: now reaches U1.8 (2)
- net U1_2: now also J5.3 (Pin_3)
- net U1_3: now reaches U1.9 (3)
- net U1_3: now also J5.4 (Pin_4)
Other:
- moved on the sheet: J6, J7, J8

Commit message: schematic done
Connections:
- net U3_0: now reaches J7.1 (Pin_1)
- net U3_0: now also U3.16 (0)
- net U3_9: now reaches J7.10 (Pin_10)
- net U3_9: now also U3.2 (9)
- net U3_1: now reaches J7.2 (Pin_2)
- net U3_1: now also U3.15 (1)
- net U3_2: now reaches J7.3 (Pin_3)
- net U3_2: now also U3.8 (2)
- net U3_3: now reaches J7.4 (Pin_4)
- net U3_3: now also U3.9 (3)
- net U3_4: now reaches J7.5 (Pin_5)
- net U3_4: now also U3.13 (4)
- net U3_5: now reaches J7.6 (Pin_6)
- net U3_5: now also U3.14 (5)
- net U3_6: now reaches J7.7 (Pin_7)
- net U3_6: now also U3.11 (6)
- net U3_7: now reaches J7.8 (Pin_8)
- net U3_7: now also U3.10 (7)
- net U3_8: now reaches J7.9 (Pin_9)
- net U3_8: now also U3.1 (8)
- net U2_8: now reaches U2.1 (8)
- net U2_8: now also J6.9 (Pin_9)
- net U2_7: now reaches U2.10 (7)
- net U2_7: now also J6.8 (Pin_8)
- net U2_6: now reaches U2.11 (6)
- net U2_6: now also J6.7 (Pin_7)
- net U2_4: now reaches U2.13 (4)
- net U2_4: now also J6.5 (Pin_5)
- net U2_5: now reaches U2.14 (5)
- net U2_5: now also J6.6 (Pin_6)
- net U2_1: now reaches U2.15 (1)
- net U2_1: now also J6.2 (Pin_2)
- net U2_0: now reaches U2.16 (0)
- net U2_0: now also J6.1 (Pin_1)
- net U2_9: now reaches U2.2 (9)
- net U2_9: now also J6.10 (Pin_10)
- net U2_2: now reaches U2.8 (2)
- net U2_2: now also J6.3 (Pin_3)
- net U2_3: now reaches U2.9 (3)
- net U2_3: now also J6.4 (Pin_4)
- net U4_0: now reaches J8.1 (Pin_1)
- net U4_0: now also U4.16 (0)
- net U4_9: now reaches J8.10 (Pin_10)
- net U4_9: now also U4.2 (9)
- net U4_1: now reaches J8.2 (Pin_2)
- net U4_1: now also U4.15 (1)
- net U4_2: now reaches J8.3 (Pin_3)
- net U4_2: now also U4.8 (2)
- net U4_3: now reaches J8.4 (Pin_4)
- net U4_3: now also U4.9 (3)
- net U4_4: now reaches J8.5 (Pin_5)
- net U4_4: now also U4.13 (4)
- net U4_5: now reaches J8.6 (Pin_6)
- net U4_5: now also U4.14 (5)
- net U4_6: now reaches J8.7 (Pin_7)
- net U4_6: now also U4.11 (6)
- net U4_7: now reaches J8.8 (Pin_8)
- net U4_7: now also U4.10 (7)
- net U4_8: now reaches J8.9 (Pin_9)
- net U4_8: now also U4.1 (8)

Commit message: new PCB
Parts:
- removed J10, J11, J12, J9: Screw_Terminal_01x02, symbol Connector:Screw_Terminal_01x02
- removed J5, J6, J7, J8: Conn_01x11_Pin, Connector_PinSocket_2.54mm:PinSocket_1x11_P2.54mm_Vertical, symbol Connector:Conn_01x11_Pin
- added J14, J17, J18, J21, J22, J25, J6, J8: Anode, Connector_PinSocket_2.54mm:PinSocket_1x02_P2.54mm_Vertical, symbol Connector:Conn_01x02_Socket
- added J15, J16, J19, J20, J23, J24, J5, J7: Number IO, Connector_PinSocket_2.54mm:PinSocket_1x05_P2.54mm_Vertical, symbol Connector:Conn_01x05_Socket
- added R1, R2, R3, R4: 12K 1W, Resistor_THT:R_Axial_DIN0414_L11.9mm_D4.5mm_P20.32mm_Horizontal, symbol Device:R_US
- C1, C2, C3, C4: footprint (none) -> Capacitor_SMD:C_0805_2012Metric_Pad1.18x1.45mm_HandSolder
- C7: footprint (none) -> Capacitor_THT:CP_Radial_D8.0mm_P3.50mm
- J1: footprint (none) -> Connector_USB:USB_Micro-B_Amphenol_10103594-0001LF_Horizontal
- J2: footprint (none) -> Connector_PinHeader_2.54mm:PinHeader_1x16_P2.54mm_Vertical
- J3: footprint (none) -> Connector_PinHeader_2.54mm:PinHeader_1x02_P2.54mm_Vertical
- J4: footprint (none) -> TerminalBlock_MetzConnect:TerminalBlock_MetzConnect_Type011_RT05502HBLC_1x02_P5.00mm_Horizontal
- U1, U2, U3, U4: footprint SN74141N:DIP762W46P254L2134H508Q16 -> Nixie_Tube_Infrastructure:DIP762W46P254L2134H508Q16
Connections:
- net 170V: now also C7.2, J3.1 (Pin_1), R1.1, R2.1, R3.1, R4.1
- net U1_0: now also J5.3 (Pin_3)
- net U1_1: now also J7.1 (Pin_1)
- net U1_2: now also J7.2 (Pin_2)
- net U1_3: now also J7.3 (Pin_3)
- net U1_4: now also J7.4 (Pin_4)
- net U1_5: now also J7.5 (Pin_5)
- net U1_6: now also J5.5 (Pin_5)
- net U1_7: now also J5.4 (Pin_4)
- net U1_8: now also J5.1 (Pin_1)
- net U1_9: now also J5.2 (Pin_2)
- net U2_0: now also J15.3 (Pin_3)
- net U2_1: now also J16.1 (Pin_1)
- net U2_2: now also J16.2 (Pin_2)
- net U2_3: now also J16.3 (Pin_3)
- net U2_4: now also J16.4 (Pin_4)
- net U2_5: now also J16.5 (Pin_5)
- net U2_6: now also J15.5 (Pin_5)
- net U2_7: now also J15.4 (Pin_4)
- net U2_8: now also J15.1 (Pin_1)
- net U2_9: now also J15.2 (Pin_2)
- net U3_0: now also J19.3 (Pin_3)
- net U3_1: now also J20.1 (Pin_1)
- net U3_2: now also J20.2 (Pin_2)
- net U3_3: now also J20.3 (Pin_3)
- net U3_4: now also J20.4 (Pin_4)
- net U3_5: now also J20.5 (Pin_5)
- net U3_6: now also J19.5 (Pin_5)
- net U3_7: now also J19.4 (Pin_4)
- net U3_8: now also J19.1 (Pin_1)
- net U3_9: now also J19.2 (Pin_2)
- net U4_0: now also J23.3 (Pin_3)
- net U4_1: now also J24.1 (Pin_1)
- net U4_2: now also J24.2 (Pin_2)
- net U4_3: now also J24.3 (Pin_3)
- net U4_4: now also J24.4 (Pin_4)
- net U4_5: now also J24.5 (Pin_5)
- net U4_6: now also J23.5 (Pin_5)
- net U4_7: now also J23.4 (Pin_4)
- net U4_8: now also J23.1 (Pin_1)
- net U4_9: now also J23.2 (Pin_2)
- new net: J18.2 (Pin_2), R3.2
- new net: J6.2 (Pin_2), R1.2
- new net: J14.2 (Pin_2), R2.2
- new net: J22.2 (Pin_2), R4.2
Other:
- moved on the sheet: J2

Commit message: updated pcb
Parts:
- J1: footprint Connector_USB:USB_Micro-B_Amphenol_10103594-0001LF_Horizontal -> Connector_USB:USB_Micro-AB_Molex_47590-0001
Changed lines of the file:
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@@
 			)
 		)
-		(property "Footprint" "Connector_USB:USB_Micro-B_Amphenol_10103594-0001LF_Horizontal"
+		(property "Footprint" "Connector_USB:USB_Micro-AB_Molex_47590-0001"
 			(at 31.75 76.2 0)
 			(effects
